File: hardware/pcb/interlock-test-coupon/interlock-test.kicad_pcb (KiCad board)
At the start: 2 copper layers, 66 x 41 mm, 18 parts, among them J1 3V3_IN, J2 MCU_CTRL, J3 CAMERA_3V3_OUT, SW1 EXTERNAL_MASTER_SWITCH, U1 MCP6547-I/P, U2 TPS22918DBVR

Commit message: refactor: 项目整体改名 AgentGlass → CodexGlasses
按需求把里面所有的名字统一换成 codex-glasses 系列：

  显示名    AgentGlass      → CodexGlasses
  标识      agent-glasses   → codex-glasses
  包名/模块 agentglass       → codexglasses
  环境变量  AGENTGLASS_*    → CODEXGLASSES_*

覆盖 93 个文本文件、约 720 处引用，以及 25 个路径：

  desktop/agentglass/                 → desktop/codexglasses/
  mobile/.../java/dev/agentglass/     → .../dev/codexglasses/
  assets/agentglass-banner.svg        → codexglasses-banner.svg
  firmware/boards/agentglass_d0.json  → codexglasses_d0.json
  hardware/.../agentglass-h1-fixture.step → codexglasses-h1-fixture.step
  releases/agentglass-*.{whl,apk}     → codexglasses-*

配套改动：
- pyproject：包名、入口脚本、package-data、license 标识
- Java：package 声明与目录一起改，AndroidManifest 里的类名同步
- Dockerfile：镜像内路径与 ENV
- wheel 重新打包（包内路径为 codexglasses/），APK 二进制未重建
  （没有 Android SDK，内部 Java 包名仍是 dev.agentglass，已在文档里注明）

另外在 README 加了「欢迎 issue 和 star」一节，说明怎么提、提什么最有用；
在 docs/evidence/README.md 写清改名对证据链的影响：源码哈希与 wheel 哈希
对应改名前那一版，APK 哈希仍然有效，不追改历史记录。

旧名残留检查：文本文件 0 处。
Other:
- board text added: "CodexGlasses LED interlock TEST ONLY / 3.3V"
- board text removed: "AgentGlass LED interlock TEST ONLY / 3.3V"
Changed lines of the file:
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@@
   (gr_line (start 68 43) (end 2 43)
     (stroke (width 0.05) (type default)) (layer "Edge.Cuts"))
-  (gr_text "AgentGlass LED interlock TEST ONLY / 3.3V" (at 35 41) (layer "F.SilkS")
+  (gr_text "CodexGlasses LED interlock TEST ONLY / 3.3V" (at 35 41) (layer "F.SilkS")
     (effects (font (size 0.8 0.8) (thickness 0.12)))
   )
