File: hardware/schematics/interlock.kicad_sch (KiCad schematic)
At the start: 18 parts, among them J1 3V3_IN, J2 MCU_CTRL, J3 CAMERA_3V3_OUT, SW1 EXTERNAL_MASTER_SWITCH, U1 MCP6547-I/P, U2 TPS22918DBVR

Commit message: refactor: 项目整体改名 AgentGlass → CodexGlasses
按需求把里面所有的名字统一换成 codex-glasses 系列：

  显示名    AgentGlass      → CodexGlasses
  标识      agent-glasses   → codex-glasses
  包名/模块 agentglass       → codexglasses
  环境变量  AGENTGLASS_*    → CODEXGLASSES_*

覆盖 93 个文本文件、约 720 处引用，以及 25 个路径：

  desktop/agentglass/                 → desktop/codexglasses/
  mobile/.../java/dev/agentglass/     → .../dev/codexglasses/
  assets/agentglass-banner.svg        → codexglasses-banner.svg
  firmware/boards/agentglass_d0.json  → codexglasses_d0.json
  hardware/.../agentglass-h1-fixture.step → codexglasses-h1-fixture.step
  releases/agentglass-*.{whl,apk}     → codexglasses-*

配套改动：
- pyproject：包名、入口脚本、package-data、license 标识
- Java：package 声明与目录一起改，AndroidManifest 里的类名同步
- Dockerfile：镜像内路径与 ENV
- wheel 重新打包（包内路径为 codexglasses/），APK 二进制未重建
  （没有 Android SDK，内部 Java 包名仍是 dev.agentglass，已在文档里注明）

另外在 README 加了「欢迎 issue 和 star」一节，说明怎么提、提什么最有用；
在 docs/evidence/README.md 写清改名对证据链的影响：源码哈希与 wheel 哈希
对应改名前那一版，APK 哈希仍然有效，不追改历史记录。

旧名残留检查：文本文件 0 处。
Parts:
- C1: symbol AgentGlass:PART_C1 -> CodexGlasses:PART_C1
- C2: symbol AgentGlass:PART_C2 -> CodexGlasses:PART_C2
- C3: symbol AgentGlass:PART_C3 -> CodexGlasses:PART_C3
- C4: symbol AgentGlass:PART_C4 -> CodexGlasses:PART_C4
- D1: symbol AgentGlass:PART_D1 -> CodexGlasses:PART_D1
- J1: symbol AgentGlass:PART_J1 -> CodexGlasses:PART_J1
- J2: symbol AgentGlass:PART_J2 -> CodexGlasses:PART_J2
- J3: symbol AgentGlass:PART_J3 -> CodexGlasses:PART_J3
- R1: symbol AgentGlass:PART_R1 -> CodexGlasses:PART_R1
- R2: symbol AgentGlass:PART_R2 -> CodexGlasses:PART_R2
- R3: symbol AgentGlass:PART_R3 -> CodexGlasses:PART_R3
- R4: symbol AgentGlass:PART_R4 -> CodexGlasses:PART_R4
- R5: symbol AgentGlass:PART_R5 -> CodexGlasses:PART_R5
- R6: symbol AgentGlass:PART_R6 -> CodexGlasses:PART_R6
- R7: symbol AgentGlass:PART_R7 -> CodexGlasses:PART_R7
- SW1: symbol AgentGlass:PART_SW1 -> CodexGlasses:PART_SW1
- U1: symbol AgentGlass:PART_U1 -> CodexGlasses:PART_U1
- U2: symbol AgentGlass:PART_U2 -> CodexGlasses:PART_U2
Changed lines of the file:
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@@
 (wire (pts (xy 102 231.27) (xy 109.84 231.27)) (stroke (width 0) (type default)))
 (label "GND" (at 102 231.27 0) (effects (font (size 1 1)) (justify left bottom)))
-(symbol (lib_id "AgentGlass:PART_J1") (at 30 30 0) (unit 1) (in_bom yes) (on_board yes)
+(symbol (lib_id "CodexGlasses:PART_J1") (at 30 30 0) (unit 1) (in_bom yes) (on_board yes)
 (property "Reference" "J1" (at 30 24.96 0) (effects (font (size 1.0 1.0))))
 (property "Value" "3V3_IN" (at 30 35.04 0) (effects (font (size 0.85 0.85))))
@@
 (pin "2")
 (instances (project "interlock" (path "/dd608bae-1de2-4c0c-948e-73c3f4dd3bfc" (reference "J1") (unit 1)))))
-(symbol (lib_id "AgentGlass:PART_SW1") (at 120 30 0) (unit 1) (in_bom yes) (on_board yes)
+(symbol (lib_id "CodexGlasses:PART_SW1") (at 120 30 0) (unit 1) (in_bom yes) (on_board yes)
 (property "Reference" "SW1" (at 120 24.96 0) (effects (font (size 1.0 1.0))))
 (property "Value" "EXTERNAL_MASTER_SWITCH" (at 120 35.04 0) (effects (font (size 0.85 0.85))))
@@
 (pin "2")
 (instances (project "interlock" (path "/dd608bae-1de2-4c0c-948e-73c3f4dd3bfc" (reference "SW1") (unit 1)))))
-(symbol (lib_id "AgentGlass:PART_J2") (at 210 30 0) (unit 1) (in_bom yes) (on_board yes)
+(symbol (lib_id "CodexGlasses:PART_J2") (at 210 30 0) (unit 1) (in_bom yes) (on_board yes)
 (property "Reference" "J2" (at 210 23.69 0) (effects (font (size 1.0 1.0))))
 (property "Value" "MCU_CTRL" (at 210 36.31 0) (effects (font (size 0.85 0.85))))
@@
 (pin "3")
 (instances (project "interlock" (path "/dd608bae-1de2-4c0c-948e-73c3f4dd3bfc" (reference "J2") (unit 1)))))
-(symbol (lib_id "AgentGlass:PART_J3") (at 300 30 0) (unit 1) (in_bom yes) (on_board yes)
+(symbol (lib_id "CodexGlasses:PART_J3") (at 300 30 0) (unit 1) (in_bom yes) (on_board yes)
 (property "Reference" "J3" (at 300 24.96 0) (effects (font (size 1.0 1.0))))
 (property "Value" "CAMERA_3V3_OUT" (at 300 35.04 0) (effects (font (size 0.85 0.85))))
@@
 (pin "2")
 (instances (project "interlock" (path "/dd608bae-1de2-4c0c-948e-73c3f4dd3bfc" (reference "J3") (unit 1)))))
-(symbol (lib_id "AgentGlass:PART_U1") (at 30 80 0) (unit 1) (in_bom yes) (on_board yes)
+(symbol (lib_id "CodexGlasses:PART_U1") (at 30 80 0) (unit 1) (in_bom yes) (on_board yes)
 (property "Reference" "U1" (at 30 67.34 0) (effects (font (size 1.0 1.0))))
 (property "Value" "MCP6547-I/P" (at 30 92.66 0) (effects (font (size 0.85 0.85))))
@@
 (pin "8")
 (instances (project "interlock" (path "/dd608bae-1de2-4c0c-948e-73c3f4dd3bfc" (reference "U1") (unit 1)))))
-(symbol (lib_id "AgentGlass:PART_U2") (at 120 80 0) (unit 1) (in_bom yes) (on_board yes)
+(symbol (lib_id "CodexGlasses:PART_U2") (at 120 80 0) (unit 1) (in_bom yes) (on_board yes)
 (property "Reference" "U2" (at 120 69.88 0) (effects (font (size 1.0 1.0))))
 (property "Value" "TPS22918DBVR" (at 120 90.12 0) (effects (font (size 0.85 0.85))))
@@
 (pin "6")
 (instances (project "interlock" (path "/dd608bae-1de2-4c0c-948e-73c3f4dd3bfc" (reference "U2") (unit 1)))))
-(symbol (lib_id "AgentGlass:PART_R1") (at 210 80 0) (unit 1) (in_bom yes) (on_board yes)
+(symbol (lib_id "CodexGlasses:PART_R1") (at 210 80 0) (unit 1) (in_bom yes) (on_board yes)
 (property "Reference" "R1" (at 210 74.96 0) (effects (font (size 1.0 1.0))))
 (property "Value" "330" (at 210 85.04 0) (effects (font (size 0.85 0.85))))
@@
 (pin "2")
 (instances (project "interlock" (path "/dd608bae-1de2-4c0c-948e-73c3f4dd3bfc" (reference "R1") (unit 1)))))
-(symbol (lib_id "AgentGlass:PART_D1") (at 300 80 0) (unit 1) (in_bom yes) (on_board yes)
+(symbol (lib_id "CodexGlasses:PART_D1") (at 300 80 0) (unit 1) (in_bom yes) (on_board yes)
 (property "Reference" "D1" (at 300 74.96 0) (effects (font (size 1.0 1.0))))
 (property "Value" "VISIBLE_GREEN_LED" (at 300 85.04 0) (effects (font (size 0.85 0.85))))
@@
 (pin "2")
 (instances (project "interlock" (path "/dd608bae-1de2-4c0c-948e-73c3f4dd3bfc" (reference "D1") (unit 1)))))
-(symbol (lib_id "AgentGlass:PART_R2") (at 30 130 0) (unit 1) (in_bom yes) (on_board yes)
+(symbol (lib_id "CodexGlasses:PART_R2") (at 30 130 0) (unit 1) (in_bom yes) (on_board yes)
 (property "Reference" "R2" (at 30 124.96 0) (effects (font (size 1.0 1.0))))
 (property "Value" "232k 1%" (at 30 135.04 0) (effects (font (size 0.85 0.85))))
@@
 (pin "2")
 (instances (project "interlock" (path "/dd608bae-1de2-4c0c-948e-73c3f4dd3bfc" (reference "R2") (unit 1)))))
-(symbol (lib_id "AgentGlass:PART_R3") (at 120 130 0) (unit 1) (in_bom yes) (on_board yes)
+(symbol (lib_id "CodexGlasses:PART_R3") (at 120 130 0) (unit 1) (in_bom yes) (on_board yes)
 (property "Reference" "R3" (at 120 124.96 0) (effects (font (size 1.0 1.0))))
 (property "Value" "100k 1%" (at 120 135.04 0) (effects (font (size 0.85 0.85))))
@@
 (pin "2")
 (instances (project "interlock" (path "/dd608bae-1de2-4c0c-948e-73c3f4dd3bfc" (reference "R3") (unit 1)))))
-(symbol (lib_id "AgentGlass:PART_R4") (at 210 130 0) (unit 1) (in_bom yes) (on_board yes)
+(symbol (lib_id "CodexGlasses:PART_R4") (at 210 130 0) (unit 1) (in_bom yes) (on_board yes)
 (property "Reference" "R4" (at 210 124.96 0) (effects (font (size 1.0 1.0))))
 (property "Value" "22.1k 1%" (at 210 135.04 0) (effects (font (size 0.85 0.85))))
@@
 (pin "2")
 (instances (project "interlock" (path "/dd608bae-1de2-4c0c-948e-73c3f4dd3bfc" (reference "R4") (unit 1)))))
-(symbol (lib_id "AgentGlass:PART_R5") (at 300 130 0) (unit 1) (in_bom yes) (on_board yes)
+(symbol (lib_id "CodexGlasses:PART_R5") (at 300 130 0) (unit 1) (in_bom yes) (on_board yes)
 (property "Reference" "R5" (at 300 124.96 0) (effects (font (size 1.0 1.0))))
 (property "Value" "100k 1%" (at 300 135.04 0) (effects (font (size 0.85 0.85))))
@@
 (pin "2")
 (instances (project "interlock" (path "/dd608bae-1de2-4c0c-948e-73c3f4dd3bfc" (reference "R5") (unit 1)))))
-(symbol (lib_id "AgentGlass:PART_R6") (at 30 180 0) (unit 1) (in_bom yes) (on_board yes)
+(symbol (lib_id "CodexGlasses:PART_R6") (at 30 180 0) (unit 1) (in_bom yes) (on_board yes)
 (property "Reference" "R6" (at 30 174.96 0) (effects (font (size 1.0 1.0))))
 (property "Value" "10k" (at 30 185.04 0) (effects (font (size 0.85 0.85))))
@@
 (pin "2")
 (instances (project "interlock" (path "/dd608bae-1de2-4c0c-948e-73c3f4dd3bfc" (reference "R6") (unit 1)))))
-(symbol (lib_id "AgentGlass:PART_R7") (at 120 180 0) (unit 1) (in_bom yes) (on_board yes)
+(symbol (lib_id "CodexGlasses:PART_R7") (at 120 180 0) (unit 1) (in_bom yes) (on_board yes)
 (property "Reference" "R7" (at 120 174.96 0) (effects (font (size 1.0 1.0))))
 (property "Value" "100k" (at 120 185.04 0) (effects (font (size 0.85 0.85))))
@@
 (pin "2")
 (instances (project "interlock" (path "/dd608bae-1de2-4c0c-948e-73c3f4dd3bfc" (reference "R7") (unit 1)))))
-(symbol (lib_id "AgentGlass:PART_C1") (at 210 180 0) (unit 1) (in_bom yes) (on_board yes)
+(symbol (lib_id "CodexGlasses:PART_C1") (at 210 180 0) (unit 1) (in_bom yes) (on_board yes)
 (property "Reference" "C1" (at 210 174.96 0) (effects (font (size 1.0 1.0))))
 (property "Value" "1uF" (at 210 185.04 0) (effects (font (size 0.85 0.85))))
@@
 (pin "2")
 (instances (project "interlock" (path "/dd608bae-1de2-4c0c-948e-73c3f4dd3bfc" (reference "C1") (unit 1)))))
-(symbol (lib_id "AgentGlass:PART_C2") (at 300 180 0) (unit 1) (in_bom yes) (on_board yes)
+(symbol (lib_id "CodexGlasses:PART_C2") (at 300 180 0) (unit 1) (in_bom yes) (on_board yes)
 (property "Reference" "C2" (at 300 174.96 0) (effects (font (size 1.0 1.0))))
 (property "Value" "1uF" (at 300 185.04 0) (effects (font (size 0.85 0.85))))
@@
 (pin "2")
 (instances (project "interlock" (path "/dd608bae-1de2-4c0c-948e-73c3f4dd3bfc" (reference "C2") (unit 1)))))
-(symbol (lib_id "AgentGlass:PART_C3") (at 30 230 0) (unit 1) (in_bom yes) (on_board yes)
+(symbol (lib_id "CodexGlasses:PART_C3") (at 30 230 0) (unit 1) (in_bom yes) (on_board yes)
 (property "Reference" "C3" (at 30 224.96 0) (effects (font (size 1.0 1.0))))
 (property "Value" "1nF" (at 30 235.04 0) (effects (font (size 0.85 0.85))))
@@
 (pin "2")
 (instances (project "interlock" (path "/dd608bae-1de2-4c0c-948e-73c3f4dd3bfc" (reference "C3") (unit 1)))))
-(symbol (lib_id "AgentGlass:PART_C4") (at 120 230 0) (unit 1) (in_bom yes) (on_board yes)
+(symbol (lib_id "CodexGlasses:PART_C4") (at 120 230 0) (unit 1) (in_bom yes) (on_board yes)
 (property "Reference" "C4" (at 120 224.96 0) (effects (font (size 1.0 1.0))))
 (property "Value" "100nF" (at 120 235.04 0) (effects (font (size 0.85 0.85))))
